Commit message: I changed the bot description

File: clean_bot_description/urdf/lidar.xacro (robot description, xacro)
@@ -3,8 +3,8 @@
     <joint name="laser_joint" type="fixed">
         <parent link="chassis"/>
-        <child link="laser_frame"/>
-        <origin xyz="0.1 0 0.175" rpy="0 0 0"/>
+        <child link="laser"/>
+        <origin xyz="0.15 0 0.175" rpy="0 0 0"/>
     </joint>
-    <link name="laser_frame">
+    <link name="laser">
         <visual>
             <geometry>
@@ -22,5 +22,5 @@
         </xacro:inertial_cylinder>
     </link>
-    <gazebo reference="laser_frame">
+    <gazebo reference="laser">
         <material>Gazebo/Red</material>
         <sensor name="laser" type="ray">

Commit message: Fix lidar orientation - rotate 180 degrees if USB faces back

File: clean_bot_description/urdf/lidar.xacro (robot description, xacro)
@@ -22,5 +22,7 @@
         <parent link="chassis"/>
         <child link="laser"/>
-        <origin xyz="0.15 0 0.175" rpy="0 0 0"/>
+        <!-- RPLIDAR A1 mounted with USB port facing BACK -->
+        <!-- If robot goes towards walls, try rpy="0 0 3.14159" (180 degrees) -->
+        <origin xyz="0.15 0 0.175" rpy="0 0 3.14159"/>
     </joint>
     <link name="laser">

Commit message: סובבתי את הלידאר

File: clean_bot_description/urdf/lidar.xacro (robot description, xacro)
@@ -23,6 +23,6 @@
         <child link="laser"/>
         <!-- RPLIDAR A1 mounted with USB port facing BACK -->
-        <!-- If robot goes towards walls, try rpy="0 0 3.14159" (180 degrees) -->
-        <origin xyz="0.15 0 0.175" rpy="0 0 3.14159"/>
+        <!-- Fixed: LiDAR is now mounted facing forward -->
+        <origin xyz="0.15 0 0.175" rpy="0 0 0"/>
     </joint>
     <link name="laser">

Commit message: inverted the inverted lidar

File: clean_bot_description/urdf/lidar.xacro (robot description, xacro)
@@ -22,7 +22,7 @@
         <parent link="chassis"/>
         <child link="laser"/>
-        <!-- RPLIDAR A1 mounted with USB port facing BACK -->
-        <!-- Fixed: LiDAR is now mounted facing forward -->
-        <origin xyz="0.15 0 0.175" rpy="0 0 0"/>
+        <!-- RPLIDAR A1 mounted with USB port facing BACK (physically rotated 180°) -->
+        <!-- The TF must match physical orientation! -->
+        <origin xyz="0.15 0 0.175" rpy="0 0 3.14159"/>
     </joint>
     <link name="laser">
